File: rgb_led/rgbled.brd (EAGLE design)
At the start: 35.9 x 29.2 mm, 9 parts, among them U1 R:1.9V, G,B:2.7V

Commit message: New version of rgbled
Parts:
- added RBP: 300, rcl:R0805
- added RGP: 420, rcl:R0805
- added RRP: 450, rcl:R0805
- moved PGRN 2.54 mm to (10.2, 62.2)
- moved PRED 2.54 mm to (26.0, 62.2)
Connections:
- removed net N$7: G1.N1, PBLU.1, PGRN.1, PRED.1, U$1.LL
- removed net N$9: PBLU.2, RBLU.2
- new net N$11: G1.N1, PBLU.1, PGRN.1, PRED.1, RBP.1, RGP.1, RRP.1, U$1.LL
- new net RRP: PRED.2, PRED.3, RRED.2, RRP.2
- net N$2: no longer PBLU.3, PGRN.3, PRED.3
- net N$6: now also PGRN.2, PGRN.3, RGP.2, RGRN.2; no longer PRED.2, RRED.2
- net N$8: now also PBLU.2, PBLU.3, RBLU.2, RBP.2; no longer PGRN.2, RGRN.2
Routing:
- net N$11: track 0.00 -> 91.2 mm, vias 0 -> 1
- net N$7: track 79.5 -> 0.00 mm, vias 1 -> 0
- net N$2: track 71.4 -> 8.53 mm
- net RRP: track 0.00 -> 17.5 mm
- net N$9: track 11.1 -> 0.00 mm
- net N$6: track 17.1 -> 13.5 mm, vias 1 -> 0
- net N$8: track 14.7 -> 15.9 mm, vias 1 -> 0
Other:
- board size 35.9 x 29.2 mm -> 35.9 x 26.7 mm
- board text added: "+"
- board text added: "-"
