File: rgb_led/rgbled.sch (EAGLE design)
At the start: 9 parts, among them U1 R:1.9V, G,B:2.7V

Commit message: New version of rgbled
Parts:
- added RBP: 300, rcl:R-US_R0805
- added RGP: 420, rcl:R-US_R0805
- added RRP: 450, rcl:R-US_R0805
Connections:
- removed net N$7: G1.-, PBLU.E, PGRN.E, PRED.E, U$1.LL
- removed net N$9: PBLU.S, RBLU.2
- new net N$11: G1.-, PBLU.E, PGRN.E, PRED.E, RBP.1, RGP.1, RRP.1, U$1.LL
- new net RRP: PRED.A, PRED.S, RRED.2, RRP.2
- net N$2: no longer PBLU.A, PGRN.A, PRED.A
- net N$6: now also PGRN.A, PGRN.S, RGP.2, RGRN.2; no longer PRED.S, RRED.2
- net N$8: now also PBLU.A, PBLU.S, RBLU.2, RBP.2; no longer PGRN.S, RGRN.2
Other:
- moved on the sheet: PBLU, PGRN, PRED
Changed lines of the file:
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@@
 <part name="G1" library="mattsownlib" deviceset="CR2032H" device="HORIZ"/>
 <part name="U$1" library="mattsownlib" deviceset="SWITCH-JS202011SCQN" device="SMD"/>
+<part name="RRP" library="rcl" deviceset="R-US_" device="R0805" value="450"/>
+<part name="RBP" library="rcl" deviceset="R-US_" device="R0805" value="300"/>
+<part name="RGP" library="rcl" deviceset="R-US_" device="R0805" value="420"/>
 </parts>
 <sheets>
@@
 <instance part="RBLU" gate="G$1" x="60.96" y="10.16"/>
 <instance part="RGRN" gate="G$1" x="60.96" y="17.78"/>
-<instance part="PRED" gate="G$1" x="73.66" y="27.94" rot="R180"/>
-<instance part="PBLU" gate="G$1" x="93.98" y="10.16" rot="R180"/>
-<instance part="PGRN" gate="G$1" x="83.82" y="20.32" rot="R180"/>
+<instance part="PRED" gate="G$1" x="81.28" y="35.56" rot="R180"/>
+<instance part="PBLU" gate="G$1" x="121.92" y="10.16" rot="R180"/>
+<instance part="PGRN" gate="G$1" x="101.6" y="22.86" rot="R180"/>
 <instance part="U1" gate="U1" x="43.18" y="17.78"/>
 <instance part="G1" gate="1" x="0" y="10.16" rot="R90"/>
 <instance part="U$1" gate="G$1" x="7.62" y="40.64"/>
+<instance part="RRP" gate="G$1" x="76.2" y="30.48" rot="R90"/>
+<instance part="RBP" gate="G$1" x="116.84" y="5.08" rot="R90"/>
+<instance part="RGP" gate="G$1" x="96.52" y="17.78" rot="R90"/>
 </instances>
 <busses>
@@
 <segment>
 <pinref part="U1" gate="U1" pin="ANODE"/>
-<wire x1="20.32" y1="17.78" x2="22.86" y2="17.78" width="0.1524" layer="91"/>
-<pinref part="PRED" gate="G$1" pin="A"/>
-<wire x1="73.66" y1="35.56" x2="20.32" y2="35.56" width="0.1524" layer="91"/>
-<wire x1="20.32" y1="35.56" x2="20.32" y2="17.78" width="0.1524" layer="91"/>
-<pinref part="PBLU" gate="G$1" pin="A"/>
-<wire x1="73.66" y1="35.56" x2="83.82" y2="35.56" width="0.1524" layer="91"/>
-<wire x1="83.82" y1="35.56" x2="93.98" y2="35.56" width="0.1524" layer="91"/>
-<wire x1="93.98" y1="35.56" x2="93.98" y2="17.78" width="0.1524" layer="91"/>
-<junction x="73.66" y="35.56"/>
-<pinref part="PGRN" gate="G$1" pin="A"/>
-<wire x1="83.82" y1="35.56" x2="83.82" y2="27.94" width="0.1524" layer="91"/>
-<junction x="83.82" y="35.56"/>
 <wire x1="15.24" y1="22.86" x2="15.24" y2="17.78" width="0.1524" layer="91"/>
-<wire x1="15.24" y1="17.78" x2="20.32" y2="17.78" width="0.1524" layer="91"/>
-<junction x="20.32" y="17.78"/>
+<wire x1="15.24" y1="17.78" x2="22.86" y2="17.78" width="0.1524" layer="91"/>
 <pinref part="U$1" gate="G$1" pin="CL"/>
 <wire x1="7.62" y1="33.02" x2="7.62" y2="22.86" width="0.1524" layer="91"/>
@@
 </segment>
 </net>
-<net name="N$7" class="0">
-<segment>
-<wire x1="0" y1="5.08" x2="0" y2="0" width="0.1524" layer="91"/>
-<wire x1="0" y1="0" x2="10.16" y2="0" width="0.1524" layer="91"/>
-<pinref part="PBLU" gate="G$1" pin="E"/>
-<wire x1="10.16" y1="0" x2="73.66" y2="0" width="0.1524" layer="91"/>
-<wire x1="73.66" y1="0" x2="83.82" y2="0" width="0.1524" layer="91"/>
-<wire x1="83.82" y1="0" x2="93.98" y2="0" width="0.1524" layer="91"/>
-<wire x1="93.98" y1="0" x2="93.98" y2="2.54" width="0.1524" layer="91"/>
-<pinref part="PRED" gate="G$1" pin="E"/>
-<wire x1="73.66" y1="20.32" x2="73.66" y2="0" width="0.1524" layer="91"/>
-<junction x="73.66" y="0"/>
-<pinref part="PGRN" gate="G$1" pin="E"/>
-<wire x1="83.82" y1="12.7" x2="83.82" y2="0" width="0.1524" layer="91"/>
-<junction x="83.82" y="0"/>
-<pinref part="G1" gate="1" pin="-"/>
-<pinref part="U$1" gate="G$1" pin="LL"/>
-<wire x1="10.16" y1="33.02" x2="10.16" y2="0" width="0.1524" layer="91"/>
-<junction x="10.16" y="0"/>
-</segment>
-</net>
-<net name="N$9" class="0">
-<segment>
-<pinref part="RBLU" gate="G$1" pin="2"/>
-<pinref part="PBLU" gate="G$1" pin="S"/>
-<wire x1="66.04" y1="10.16" x2="88.9" y2="10.16" width="0.1524" layer="91"/>
-</segment>
-</net>
-<net name="N$6" class="0">
-<segment>
-<pinref part="RRED" gate="G$1" pin="2"/>
-<pinref part="PRED" gate="G$1" pin="S"/>
-<wire x1="66.04" y1="25.4" x2="68.58" y2="25.4" width="0.1524" layer="91"/>
-<wire x1="68.58" y1="25.4" x2="68.58" y2="27.94" width="0.1524" layer="91"/>
-</segment>
-</net>
-<net name="N$8" class="0">
-<segment>
-<pinref part="RGRN" gate="G$1" pin="2"/>
-<pinref part="PGRN" gate="G$1" pin="S"/>
-<wire x1="66.04" y1="17.78" x2="78.74" y2="17.78" width="0.1524" layer="91"/>
-<wire x1="78.74" y1="17.78" x2="78.74" y2="20.32" width="0.1524" layer="91"/>
-</segment>
-</net>
 <net name="N$10" class="0">
 <segment>
@@
 </segment>
 </net>
+<net name="RRP" class="0">
+<segment>
+<pinref part="PRED" gate="G$1" pin="S"/>
+<pinref part="RRP" gate="G$1" pin="2"/>
+<pinref part="RRED" gate="G$1" pin="2"/>
+<wire x1="66.04" y1="25.4" x2="76.2" y2="35.56" width="0.1524" layer="91"/>
+<junction x="76.2" y="35.56"/>
+<pinref part="PRED" gate="G$1" pin="A"/>
+<wire x1="76.2" y1="35.56" x2="76.2" y2="43.18" width="0.1524" layer="91"/>
+<wire x1="76.2" y1="43.18" x2="81.28" y2="43.18" width="0.1524" layer="91"/>
+</segment>
+</net>
+<net name="N$6" class="0">
+<segment>
+<pinref part="PGRN" gate="G$1" pin="S"/>
+<pinref part="RGP" gate="G$1" pin="2"/>
+<pinref part="PGRN" gate="G$1" pin="A"/>
+<wire x1="96.52" y1="22.86" x2="96.52" y2="30.48" width="0.1524" layer="91"/>
+<wire x1="96.52" y1="30.48" x2="101.6" y2="30.48" width="0.1524" layer="91"/>
+<junction x="96.52" y="22.86"/>
+<pinref part="RGRN" gate="G$1" pin="2"/>
+<wire x1="66.04" y1="17.78" x2="91.44" y2="17.78" width="0.1524" layer="91"/>
+<wire x1="91.44" y1="17.78" x2="96.52" y2="22.86" width="0.1524" layer="91"/>
+</segment>
+</net>
+<net name="N$8" class="0">
+<segment>
+<pinref part="PBLU" gate="G$1" pin="S"/>
+<pinref part="RBP" gate="G$1" pin="2"/>
+<pinref part="PBLU" gate="G$1" pin="A"/>
+<wire x1="116.84" y1="10.16" x2="116.84" y2="17.78" width="0.1524" layer="91"/>
+<wire x1="116.84" y1="17.78" x2="121.92" y2="17.78" width="0.1524" layer="91"/>
+<junction x="116.84" y="10.16"/>
+<pinref part="RBLU" gate="G$1" pin="2"/>
+<wire x1="66.04" y1="10.16" x2="116.84" y2="10.16" width="0.1524" layer="91"/>
+</segment>
+</net>
+<net name="N$11" class="0">
+<segment>
+<pinref part="RGP" gate="G$1" pin="1"/>
+<pinref part="PGRN" gate="G$1" pin="E"/>
+<wire x1="96.52" y1="12.7" x2="99.06" y2="12.7" width="0.1524" layer="91"/>
+<wire x1="99.06" y1="12.7" x2="101.6" y2="15.24" width="0.1524" layer="91"/>
+<pinref part="RRP" gate="G$1" pin="1"/>
+<pinref part="PRED" gate="G$1" pin="E"/>
+<wire x1="76.2" y1="25.4" x2="78.74" y2="25.4" width="0.1524" layer="91"/>
+<wire x1="78.74" y1="25.4" x2="81.28" y2="27.94" width="0.1524" layer="91"/>
+<wire x1="0" y1="5.08" x2="0" y2="0" width="0.1524" layer="91"/>
+<wire x1="0" y1="0" x2="10.16" y2="0" width="0.1524" layer="91"/>
+<wire x1="10.16" y1="0" x2="76.2" y2="0" width="0.1524" layer="91"/>
+<pinref part="G1" gate="1" pin="-"/>
+<pinref part="U$1" gate="G$1" pin="LL"/>
+<wire x1="10.16" y1="33.02" x2="10.16" y2="0" width="0.1524" layer="91"/>
+<junction x="10.16" y="0"/>
+<wire x1="76.2" y1="25.4" x2="76.2" y2="0" width="0.1524" layer="91"/>
+<junction x="76.2" y="25.4"/>
+<junction x="76.2" y="0"/>
+<pinref part="RBP" gate="G$1" pin="1"/>
+<pinref part="PBLU" gate="G$1" pin="E"/>
+<wire x1="116.84" y1="0" x2="119.38" y2="0" width="0.1524" layer="91"/>
+<wire x1="119.38" y1="0" x2="121.92" y2="2.54" width="0.1524" layer="91"/>
+<wire x1="76.2" y1="0" x2="96.52" y2="0" width="0.1524" layer="91"/>
+<junction x="116.84" y="0"/>
+<wire x1="96.52" y1="0" x2="116.84" y2="0" width="0.1524" layer="91"/>
+<wire x1="96.52" y1="12.7" x2="96.52" y2="0" width="0.1524" layer="91"/>
+<junction x="96.52" y="12.7"/>
+<junction x="96.52" y="0"/>
+</segment>
+</net>
